Commit message: Starting the process of adding gazebo tags for gazebo simulation

File: mico_description/urdf/mico_arm.urdf.xacro (robot description, xacro)
@@ -142,4 +142,23 @@
 		</link>
 	</xacro:macro>
+	<xacro:macro name="mico_joint_transmission" params="transmission_name joint_name motor_name">
+		<transmission name="${transmission_name}">
+			<type>transmission_interface/SimpleTransmission</type>
+			<joint name="${joint_name}">
+				<hardwareInterface>EffortJointInterface</hardwareInterface>
+			</joint>
+			<actuator name="${motor_name}">
+			<mechanicalReduction>1</mechanicalReduction>
+			</actuator>
+		</transmission>
+	</xacro:macro>
+	<xacro:macro name="mico_joint_friction_gazebo" params="link_name mu1 mu2 kp kd">
+		<gazebo reference="${link_name}">
+			<mu1 value="${mu1}" />
+			<mu2  value="${mu2}"/>
+				<kp value="${kp}" />
+				<kd value="${kd}" />
+		</gazebo>
+	</xacro:macro>
 	<xacro:macro name="mico_joint" params="joint_name type parent child joint_axis_xyz joint_origin_xyz joint_origin_rpy lower_limit upper_limit">
 		<joint name="${joint_name}" type="${type}">

Commit message: Transmissions and friction joints for gazebo added to the mico model

File: mico_description/urdf/mico_arm.urdf.xacro (robot description, xacro)
@@ -161,4 +161,20 @@
 		</gazebo>
 	</xacro:macro>
+	<xacro:property name="mu1_default" value="0.2" />
+	<xacro:property name="mu2_default" value="0.2" />
+	<xacro:property name="kp_default" value="1000000.0" />
+	<xacro:property name="kd_default" value="1.0" />
+	<xacro:mico_joint_transmission transmission_name="${joint_1}_transmission" joint_name="${joint_1}" motor_name="${joint_1}_motor"/>
+	<xacro:mico_joint_transmission transmission_name="${joint_2}_transmission" joint_name="${joint_2}" motor_name="${joint_2}_motor"/>
+	<xacro:mico_joint_transmission transmission_name="${joint_3}_transmission" joint_name="${joint_3}" motor_name="${joint_3}_motor"/>
+	<xacro:mico_joint_transmission transmission_name="${joint_4}_transmission" joint_name="${joint_4}" motor_name="${joint_4}_motor"/>
+	<xacro:mico_joint_transmission transmission_name="${joint_5}_transmission" joint_name="${joint_5}" motor_name="${joint_5}_motor"/>
+	<xacro:mico_joint_transmission transmission_name="${joint_6}_transmission" joint_name="${joint_6}" motor_name="${joint_6}_motor"/>
+	<xacro:mico_joint_friction_gazebo link_name="${link_base}" mu1="${mu1_default}" mu2="${mu2_default}" kp="${kp_default}" kd="${kd_default}" />
+	<xacro:mico_joint_friction_gazebo link_name="${link}" mu1="${mu1_default}" mu2="${mu2_default}" kp="${kp_default}" kd="${kd_default}" />
+	<xacro:mico_joint_friction_gazebo link_name="${link_1}" mu1="${mu1_default}" mu2="${mu2_default}" kp="${kp_default}" kd="${kd_default}" />
+	<xacro:mico_joint_friction_gazebo link_name="${link_2}" mu1="${mu1_default}" mu2="${mu2_default}" kp="${kp_default}" kd="${kd_default}" />
+	<xacro:mico_joint_friction_gazebo link_name="${link_3}" mu1="${mu1_default}" mu2="${mu2_default}" kp="${kp_default}" kd="${kd_default}" />
+	<xacro:mico_joint_friction_gazebo link_name="${link_hand}" mu1="${mu1_default}" mu2="${mu2_default}" kp="${kp_default}" kd="${kd_default}" />
 	<xacro:macro name="mico_joint" params="joint_name type parent child joint_axis_xyz joint_origin_xyz joint_origin_rpy lower_limit upper_limit">
 		<joint name="${joint_name}" type="${type}">

Commit message: small changes for testing

File: mico_description/urdf/mico_arm.urdf.xacro (robot description, xacro)
@@ -76,4 +76,9 @@
 	<xacro:macro name="mico_link" params="link_name">
 		<link name="${link_name}">
+	    <inertial>
+                <mass value="1"/>
+                <inertia ixx="0.1" ixy="0" ixz="0" iyy="0.1" iyz="0" izz="0.1"/>
+                <origin/>
+            </inertial>
 			<visual>
 				<geometry>
@@ -93,4 +98,9 @@
 	<xacro:macro name="mico_link_suffix" params="link_name suffix">
 		<link name="${link_name}_${suffix}">
+       	<inertial>
+                <mass value="0.25"/>
+                <inertia ixx="0.01" ixy="0" ixz="0" iyy="0.01" iyz="0" izz="0.01"/>
+                <origin/>
+            </inertial>
 			<visual>
 				<geometry>
@@ -110,4 +120,9 @@
 	<xacro:macro name="mico_link_4_5" params="link_name suffix">
 		<link name="${link_name}_${suffix}">
+	    <inertial>
+                <mass value="0.5"/>
+                <inertia ixx="0.01" ixy="0" ixz="0" iyy="0.01" iyz="0" izz="0.01"/>
+                <origin/>
+            </inertial>
 			<visual>
 				<geometry>
@@ -127,4 +142,9 @@
 	<xacro:macro name="mico_ring_cover" params="suffix size">
 		<link name="mico_${size}_ring_cover_${suffix}">
+	    <inertial>
+                <mass value="0"/>
+                <inertia ixx="0" ixy="0" ixz="0" iyy="0" iyz="0" izz="0"/>
+                <origin/>
+            </inertial>
 			<visual>
 				<geometry>
@@ -196,4 +216,10 @@
 	</xacro:macro>
 	<xacro:macro name="mico_arm" params="parent xyz rpy">
+	<gazebo>
+            <plugin filename="libgazebo_ros_control.so" name="gazebo_ros_controller_manager">
+                <!-- <robotNamespace>/</robotNamespace> -->
+                <robotParam>robot_description</robotParam>
+            </plugin>
+        </gazebo>
 		<xacro:mico_link link_name="${link_base}" />
 		<xacro:mico_joint joint_name="${joint_base}" type="fixed" parent="${parent}" child="${link_base}" joint_axis_xyz="${joint_base_axis_xyz}" joint_origin_xyz="${xyz}" joint_origin_rpy="${rpy}" lower_limit="-${J_LIM}" upper_limit="${J_LIM}" />
