Commit message: debugging simulation

File: jaco_description/urdf/jaco_arm.urdf.xacro (robot description, xacro)
@@ -196,5 +196,5 @@
             <type>transmission_interface/SimpleTransmission</type>
             <joint name="${joint_name}">
-              <hardwareInterface>PositionJointInterface</hardwareInterface>
+              <hardwareInterface>EffortJointInterface</hardwareInterface>
             </joint>
             <actuator name="${joint_name}_motor">

File: mico_description/robots/support_and_arm_gazebo.urdf.xacro (robot description, xacro)
@@ -46,5 +46,5 @@
 	<!-- 		</geometry> -->
 	<!-- 	</collision> -->
-	<!-- </link> -->
+	<!-- </link>
 	<link name="support">
         <inertial>
@@ -69,5 +69,10 @@
 	  <parent link="root" />
 	  <child link="support" />
+	</joint>-->
+	<link name="world"/>
+	<joint name="fixed" type="fixed">
+	    <parent link="world"/>
+	    <child link="root"/>
 	</joint>
-	<xacro:mico_arm parent="support" xyz="0 0 0.2" rpy="0 0 0" />
+	<xacro:mico_arm parent="root" xyz="0 0 0.2" rpy="0 0 0" />
 </robot>

File: mico_description/urdf/mico_arm.urdf.xacro (robot description, xacro)
@@ -144,5 +144,5 @@
 	    <inertial>
                 <mass value="0"/>
-                <inertia ixx="0" ixy="0" ixz="0" iyy="0" iyz="0" izz="0"/>
+                <inertia ixx="0.001" ixy="0" ixz="0" iyy="0.001" iyz="0" izz="0.001"/>
                 <origin/>
             </inertial>
@@ -173,32 +173,24 @@
 		</transmission>
 	</xacro:macro>
-	<xacro:macro name="mico_joint_friction_gazebo" params="link_name mu1 mu2 kp kd">
+	<xacro:macro name="mico_link_friction_gazebo" params="link_name mu1 mu2">
 		<gazebo reference="${link_name}">
 			<mu1 value="${mu1}" />
 			<mu2  value="${mu2}"/>
-				<kp value="${kp}" />
-				<kd value="${kd}" />
+			<selfCollide value="true" />
 		</gazebo>
 	</xacro:macro>
-	<xacro:property name="mu1_default" value="0.2" />
-	<xacro:property name="mu2_default" value="0.2" />
+	<xacro:macro name="mico_joint_params_gazebo" params="joint_name kp kd">
+		<gazebo reference="${joint_name}">
+			<kd value="${kd}" />
+			<kp value="${kp}" />
+			<stopCfm value="${kp}" />
+			<stopErp value="${kd}" />
+			<fudgeFactor value="1.0" />
+		</gazebo>
+	</xacro:macro>
+	<xacro:property name="mu1_default" value="0.7" />
+	<xacro:property name="mu2_default" value="0.7" />
 	<xacro:property name="kp_default" value="1000000.0" />
 	<xacro:property name="kd_default" value="1.0" />
-	<xacro:mico_joint_transmission transmission_name="${joint_1}_transmission" joint_name="${joint_1}" motor_name="${joint_1}_motor"/>
-	<xacro:mico_joint_transmission transmission_name="${joint_2}_transmission" joint_name="${joint_2}" motor_name="${joint_2}_motor"/>
-	<xacro:mico_joint_transmission transmission_name="${joint_3}_transmission" joint_name="${joint_3}" motor_name="${joint_3}_motor"/>
-	<xacro:mico_joint_transmission transmission_name="${joint_4}_transmission" joint_name="${joint_4}" motor_name="${joint_4}_motor"/>
-	<xacro:mico_joint_transmission transmission_name="${joint_5}_transmission" joint_name="${joint_5}" motor_name="${joint_5}_motor"/>
-	<xacro:mico_joint_transmission transmission_name="${joint_6}_transmission" joint_name="${joint_6}" motor_name="${joint_6}_motor"/>
-	<xacro:mico_joint_transmission transmission_name="${joint_finger_1}_transmission" joint_name="${joint_finger_1}" motor_name="${joint_finger_1}_motor"/>
-	<xacro:mico_joint_transmission transmission_name="${joint_finger_2}_transmission" joint_name="${joint_finger_2}" motor_name="${joint_finger_2}_motor"/>
-	<xacro:mico_joint_friction_gazebo link_name="${link_base}" mu1="${mu1_default}" mu2="${mu2_default}" kp="${kp_default}" kd="${kd_default}" />
-	<xacro:mico_joint_friction_gazebo link_name="${link}" mu1="${mu1_default}" mu2="${mu2_default}" kp="${kp_default}" kd="${kd_default}" />
-	<xacro:mico_joint_friction_gazebo link_name="${link_1}" mu1="${mu1_default}" mu2="${mu2_default}" kp="${kp_default}" kd="${kd_default}" />
-	<xacro:mico_joint_friction_gazebo link_name="${link_2}" mu1="${mu1_default}" mu2="${mu2_default}" kp="${kp_default}" kd="${kd_default}" />
-	<xacro:mico_joint_friction_gazebo link_name="${link_3}" mu1="${mu1_default}" mu2="${mu2_default}" kp="${kp_default}" kd="${kd_default}" />
-	<xacro:mico_joint_friction_gazebo link_name="${link_hand}" mu1="${mu1_default}" mu2="${mu2_default}" kp="${kp_default}" kd="${kd_default}" />
-	<xacro:mico_joint_friction_gazebo link_name="mico_link_finger_1" mu1="${mu1_default}" mu2="${mu2_default}" kp="${kp_default}" kd="${kd_default}" />
-	<xacro:mico_joint_friction_gazebo link_name="mico_link_finger_2" mu1="${mu1_default}" mu2="${mu2_default}" kp="${kp_default}" kd="${kd_default}" />
 	<xacro:macro name="mico_joint" params="joint_name type parent child joint_axis_xyz joint_origin_xyz joint_origin_rpy lower_limit upper_limit">
 		<joint name="${joint_name}" type="${type}">
@@ -221,5 +213,5 @@
 	<xacro:macro name="mico_arm" params="parent xyz rpy">
 	<gazebo>
-            <plugin filename="libgazebo_ros_control.so" name="gazebo_ros_controller_manager">
+            <plugin name="gazebo_ros_controller manager" filename="libgazebo_ros_control.so">
                 <robotNamespace>/mico_arm</robotNamespace>
                 <robotParam>robot_description</robotParam>
@@ -260,4 +252,26 @@
 		<xacro:mico_link_suffix link_name="${link_finger_tip}" suffix="2"/>
 		<xacro:mico_finger_joint joint_name="${joint_finger_tip_2}" type="fixed" parent="${link_finger}_2" child="${link_finger_tip}_2" joint_axis_xyz="${joint_finger_tip_2_axis_xyz}" joint_origin_xyz="${joint_finger_tip_2_origin_xyz}" joint_origin_rpy="${joint_finger_tip_2_origin_rpy}" lower_limit="${joint_finger_tip_2_lower_limit}" upper_limit="${joint_finger_tip_2_upper_limit}" />
+	<xacro:mico_link_friction_gazebo link_name="${link_base}" mu1="${mu1_default}" mu2="${mu2_default}" />
+	<xacro:mico_link_friction_gazebo link_name="${link}" mu1="${mu1_default}" mu2="${mu2_default}"  />
+	<xacro:mico_link_friction_gazebo link_name="${link_1}" mu1="${mu1_default}" mu2="${mu2_default}" />
+	<xacro:mico_link_friction_gazebo link_name="${link_2}" mu1="${mu1_default}" mu2="${mu2_default}" />
+	<xacro:mico_link_friction_gazebo link_name="${link_3}" mu1="${mu1_default}" mu2="${mu2_default}" />
+	<xacro:mico_link_friction_gazebo link_name="${link_hand}" mu1="${mu1_default}" mu2="${mu2_default}" />
+	<xacro:mico_link_friction_gazebo link_name="mico_link_finger_1" mu1="${mu1_default}" mu2="${mu2_default}" />
+	<xacro:mico_link_friction_gazebo link_name="mico_link_finger_2" mu1="${mu1_default}" mu2="${mu2_default}" />
+	<xacro:mico_joint_params_gazebo joint_name="${joint_1}" kp="${kp_default}" kd="${kd_default}" />
+	<xacro:mico_joint_params_gazebo joint_name="${joint_2}" kp="${kp_default}" kd="${kd_default}" />
+	<xacro:mico_joint_params_gazebo joint_name="${joint_3}" kp="${kp_default}" kd="${kd_default}" />
+	<xacro:mico_joint_params_gazebo joint_name="${joint_4}" kp="${kp_default}" kd="${kd_default}" />
+	<xacro:mico_joint_params_gazebo joint_name="${joint_5}" kp="${kp_default}" kd="${kd_default}" />
+	<xacro:mico_joint_params_gazebo joint_name="${joint_6}" kp="${kp_default}" kd="${kd_default}" />
+	<xacro:mico_joint_transmission transmission_name="${joint_1}_transmission" joint_name="${joint_1}" motor_name="${joint_1}_motor"/>
+	<xacro:mico_joint_transmission transmission_name="${joint_2}_transmission" joint_name="${joint_2}" motor_name="${joint_2}_motor"/>
+	<xacro:mico_joint_transmission transmission_name="${joint_3}_transmission" joint_name="${joint_3}" motor_name="${joint_3}_motor"/>
+	<xacro:mico_joint_transmission transmission_name="${joint_4}_transmission" joint_name="${joint_4}" motor_name="${joint_4}_motor"/>
+	<xacro:mico_joint_transmission transmission_name="${joint_5}_transmission" joint_name="${joint_5}" motor_name="${joint_5}_motor"/>
+	<xacro:mico_joint_transmission transmission_name="${joint_6}_transmission" joint_name="${joint_6}" motor_name="${joint_6}_motor"/>
+	<xacro:mico_joint_transmission transmission_name="${joint_finger_1}_transmission" joint_name="${joint_finger_1}" motor_name="${joint_finger_1}_motor"/>
+	<xacro:mico_joint_transmission transmission_name="${joint_finger_2}_transmission" joint_name="${joint_finger_2}" motor_name="${joint_finger_2}_motor"/>
 	</xacro:macro>
 </robot>
